File: Schematics/74HC/RevC3/CPU2908C3.sch (KiCad schematic (older format))
At the start: 40 parts, among them J1 Conn_02x20_Odd_Even, U1 74HC08D, U117 TC74VHCT541, U119 74HC74, U121 74AHC1G32, U2 74HC08D, U3 TC74VHCT04AFT, U4 TC74VHC574F, U6 74HC74, U7 TC74VHC574F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

Commit message: revA3
Parts:
- added unit 5 of U3
- added unit 6 of U3
- added unit 2 of U3
Connections:
- net labels added: nE, nQ
- net labels removed: ~clkE
- wire segments 343 -> 357
- no-connect marks 8 -> 9
Other:
- moved on the sheet: U3A, U3D
Changed lines of the file:
@@
 Wire Wire Line
 	2150 4500 2450 4500
-Text Label 2200 4500 0    50   ~ 0
+Text Label 2450 4500 2    50   ~ 0
 Q
 Wire Wire Line
@@
 ExBusCtrl3
 Entry Wire Line
-	3350 2950 3450 3050
-Entry Wire Line
-	3350 3050 3450 3150
+	3200 2950 3300 3050
+Entry Wire Line
+	3200 3050 3300 3150
 Wire Wire Line
 	4400 3000 4200 3000
@@
 	4350 3750 4400 3750
 Wire Wire Line
-	3450 3050 4350 3050
+	3300 3050 4350 3050
 Wire Wire Line
 	5000 3100 5200 3100
@@
 Wire Wire Line
 	2150 4300 2450 4300
-Text Label 2200 4300 0    50   ~ 0
+Text Label 2450 4300 2    50   ~ 0
 E
 Wire Bus Line
@@
 Wire Wire Line
 	2150 4600 2450 4600
-Text Label 2200 4400 0    50   ~ 0
-~clkE
-Text Label 2200 4600 0    50   ~ 0
-~clkQ
 Text Label 9700 4650 2    50   ~ 0
 D[0..7]
@@
 Wire Wire Line
 	2150 1200 2550 1200
-Text Label 2200 1000 0    50   ~ 0
+Text Label 2550 1000 2    50   ~ 0
 ~RSTO
 $Sheet
@@
 F16 "IRQH" O R 2150 1100 50
 $EndSheet
-Text Label 2200 2700 0    50   ~ 0
+Text Label 2450 2700 2    50   ~ 0
 ~Reset
-Text Label 2200 2600 0    50   ~ 0
-~clkQ
-Text Label 2200 2400 0    50   ~ 0
-~clkE
 Text Label 2450 2300 2    50   ~ 0
 E
@@
 Wire Bus Line
 	3000 1750 3000 3450
-Text Label 2200 1200 0    50   ~ 0
+Text Label 2550 1200 2    50   ~ 0
 ~IRQ
 Wire Wire Line
@@
 Wire Wire Line
 	2150 1950 2450 1950
-Text Label 2250 1850 0    50   ~ 0
+Text Label 2450 1850 2    50   ~ 0
 S0
-Text Label 2250 1950 0    50   ~ 0
+Text Label 2450 1950 2    50   ~ 0
 S1
 Wire Wire Line
 	2150 1100 2550 1100
-Text Label 2200 1100 0    50   ~ 0
+Text Label 2550 1100 2    50   ~ 0
 IRQH
 Wire Bus Line
@@
 Wire Wire Line
 	3850 2900 5200 2900
-Wire Wire Line
-	4500 6100 4550 6100
 Wire Wire Line
 	6350 3600 6350 4250
@@
 Wire Wire Line
 	5250 6000 5250 4150
-Connection ~ 3950 4900
-Wire Wire Line
-	4550 4900 3950 4900
-Wire Wire Line
-	3450 4900 3950 4900
-Wire Wire Line
-	3450 5000 3900 5000
-Text Label 3500 5000 0    50   ~ 0
+Connection ~ 3850 4900
+Wire Wire Line
+	4550 4900 3850 4900
+Wire Wire Line
+	3300 4900 3850 4900
+Wire Wire Line
+	3300 5000 3800 5000
+Text Label 3350 5000 0    50   ~ 0
 ExBusCtrl1
-Text Label 3500 4900 0    50   ~ 0
+Text Label 3350 4900 0    50   ~ 0
 ExBusCtrl0
 Entry Wire Line
-	3350 4900 3450 5000
-Entry Wire Line
-	3350 4800 3450 4900
+	3200 4900 3300 5000
+Entry Wire Line
+	3200 4800 3300 4900
 Wire Wire Line
 	6350 3600 6900 3600
@@
 Connection ~ 6600 4700
 Wire Wire Line
-	10600 5100 10150 5100
-Wire Wire Line
-	10150 5100 10150 4700
-$Comp
-L power:+5V #PWR08
-U 1 1 6F4D3D76
-P 10150 4700
-F 0 "#PWR08" H 10150 4550 50  0001 C CNN
-F 1 "+5V" H 10165 4873 50  0000 C CNN
-F 2 "" H 10150 4700 50  0001 C CNN
-F 3 "" H 10150 4700 50  0001 C CNN
-	1    10150 4700
-	1    0    0    -1
-$EndComp
+	10600 5100 10250 5100
 $Comp
 L CPU2908CLocal:74HC125 U8
@@
 Wire Wire Line
 	7600 800  7850 800
-Text Label 4000 800  2    50   ~ 0
-~clkE
 Wire Wire Line
 	3750 800  4000 800
-Text Label 5350 800  2    50   ~ 0
-~clkQ
 Wire Wire Line
 	5100 800  5350 800
@@
 L CPU2908CLocal:74HC04 U?
 U 1 1 5F06C858
-P 7350 800
+P 3500 800
 AR Path="/5DC31740/5F06C858" Ref="U?"  Part="1"
 AR Path="/5F06C858" Ref="U3"  Part="1"
-F 0 "U3" H 7350 1075 50  0000 C CNN
-F 1 "TC74VHCT04AFT" H 7350 984 50  0000 C CNN
-F 2 "Housings_SSOP:TSSOP-14_4.4x5mm_Pitch0.65mm" H 7250 800 50  0001 C CNN
-F 3 "http://akizukidenshi.com/download/ds/toshiba/TC74VHCT04AFT.pdf" H 7250 800 50  0001 C CNN
-	1    7350 800
+F 0 "U3" H 3500 1075 50  0000 C CNN
+F 1 "TC74VHCT04AFT" H 3500 984 50  0000 C CNN
+F 2 "Housings_SSOP:TSSOP-14_4.4x5mm_Pitch0.65mm" H 3400 800 50  0001 C CNN
+F 3 "http://akizukidenshi.com/download/ds/toshiba/TC74VHCT04AFT.pdf" H 3400 800 50  0001 C CNN
+	1    3500 800
 	1    0    0    -1
 $EndComp
@@
 $EndComp
 Wire Wire Line
-	3450 3150 4300 3150
+	3300 3150 4300 3150
 Wire Wire Line
 	4350 3050 4350 3750
@@
 	5350 3650 5350 3000
 Wire Bus Line
-	3050 2800 3350 2800
+	3050 2800 3200 2800
 $Comp
 L Device:R R?
@@
 L CPU2908CLocal:74HC04 U?
 U 4 1 5F08D35A
-P 3500 800
+P 4200 6900
 AR Path="/5DC31740/5F08D35A" Ref="U?"  Part="1"
 AR Path="/5F08D35A" Ref="U3"  Part="4"
-F 0 "U3" H 3500 1075 50  0000 C CNN
-F 1 "TC74VHCT04AFT" H 3500 984 50  0000 C CNN
-F 2 "Housings_SSOP:TSSOP-14_4.4x5mm_Pitch0.65mm" H 3400 800 50  0001 C CNN
-F 3 "http://akizukidenshi.com/download/ds/toshiba/TC74VHCT04AFT.pdf" H 3400 800 50  0001 C CNN
-	4    3500 800
+F 0 "U3" H 4200 7175 50  0000 C CNN
+F 1 "TC74VHCT04AFT" H 4200 7084 50  0000 C CNN
+F 2 "Housings_SSOP:TSSOP-14_4.4x5mm_Pitch0.65mm" H 4100 6900 50  0001 C CNN
+F 3 "http://akizukidenshi.com/download/ds/toshiba/TC74VHCT04AFT.pdf" H 4100 6900 50  0001 C CNN
+	4    4200 6900
 	1    0    0    -1
 $EndComp
@@
 $EndComp
 Wire Wire Line
-	4050 4500 3950 4500
-Wire Wire Line
-	3950 4500 3950 4900
-Wire Wire Line
-	4050 4400 3900 4400
-Wire Wire Line
-	3900 4400 3900 5000
+	4050 4500 3850 4500
+Wire Wire Line
+	3850 4500 3850 4900
+Wire Wire Line
+	4050 4400 3800 4400
+Wire Wire Line
+	3800 4400 3800 5000
 Wire Wire Line
 	4600 4450 4800 4450
@@
 	6050 4250 6350 4250
 NoConn ~ 10850 4850
-Wire Wire Line
-	10250 4850 10250 5250
 $Comp
 L Device:R R?
@@
 NoConn ~ 2700 4150
 NoConn ~ 10400 2300
+Wire Wire Line
+	3800 5000 4000 5000
+Wire Wire Line
+	4000 5000 4000 5100
+Wire Wire Line
+	4000 5100 4550 5100
+Connection ~ 3800 5000
+$Comp
+L CPU2908CLocal:74HC04 U?
+U 5 1 62843F9A
+P 4200 6100
+AR Path="/5DC31740/62843F9A" Ref="U?"  Part="1"
+AR Path="/62843F9A" Ref="U3"  Part="5"
+F 0 "U3" H 4200 6375 50  0000 C CNN
+F 1 "TC74VHCT04AFT" H 4200 5950 50  0000 C CNN
+F 2 "Housings_SSOP:TSSOP-14_4.4x5mm_Pitch0.65mm" H 4100 6100 50  0001 C CNN
+F 3 "http://akizukidenshi.com/download/ds/toshiba/TC74VHCT04AFT.pdf" H 4100 6100 50  0001 C CNN
+	5    4200 6100
+	1    0    0    -1
+$EndComp
+Wire Wire Line
+	4450 6100 4550 6100
+Wire Wire Line
+	3850 4900 3850 6100
+Wire Wire Line
+	3850 6100 3950 6100
+Wire Wire Line
+	3800 5900 4550 5900
+$Comp
+L CPU2908CLocal:74HC04 U?
+U 6 1 6297AD32
+P 4200 7550
+AR Path="/5DC31740/6297AD32" Ref="U?"  Part="1"
+AR Path="/6297AD32" Ref="U3"  Part="6"
+F 0 "U3" H 4200 7825 50  0000 C CNN
+F 1 "TC74VHCT04AFT" H 4200 7400 50  0000 C CNN
+F 2 "Housings_SSOP:TSSOP-14_4.4x5mm_Pitch0.65mm" H 4100 7550 50  0001 C CNN
+F 3 "http://akizukidenshi.com/download/ds/toshiba/TC74VHCT04AFT.pdf" H 4100 7550 50  0001 C CNN
+	6    4200 7550
+	1    0    0    -1
+$EndComp
+Wire Wire Line
+	4450 6900 4550 6900
+Wire Wire Line
+	3800 5900 3800 6900
+Wire Wire Line
+	3800 6900 3950 6900
+Connection ~ 3800 5900
+Wire Wire Line
+	3850 6100 3850 7100
+Wire Wire Line
+	3850 7100 4550 7100
+Connection ~ 3850 6100
+Wire Wire Line
+	3800 5000 3800 5900
+$Comp
+L CPU2908CLocal:74HC04 U?
+U 2 1 633036F5
+P 7350 800
+AR Path="/5DC31E28/633036F5" Ref="U?"  Part="2"
+AR Path="/633036F5" Ref="U3"  Part="2"
+F 0 "U3" H 7350 1075 50  0000 C CNN
+F 1 "TC74VHCT04AFT" H 7350 984 50  0000 C CNN
+F 2 "Housings_SSOP:TSSOP-14_4.4x5mm_Pitch0.65mm" H 7250 800 50  0001 C CNN
+F 3 "http://akizukidenshi.com/download/ds/toshiba/TC74VHCT04AFT.pdf" H 7250 800 50  0001 C CNN
+	2    7350 800
+	1    0    0    -1
+$EndComp
+$Comp
+L power:+5V #PWR0105
+U 1 1 63331C36
+P 3750 7500
+F 0 "#PWR0105" H 3750 7350 50  0001 C CNN
+F 1 "+5V" H 3765 7673 50  0000 C CNN
+F 2 "" H 3750 7500 50  0001 C CNN
+F 3 "" H 3750 7500 50  0001 C CNN
+	1    3750 7500
+	1    0    0    -1
+$EndComp
+Wire Wire Line
+	3750 7500 3750 7550
+Wire Wire Line
+	3750 7550 3950 7550
+NoConn ~ 4450 7550
+Wire Wire Line
+	10250 4850 10250 5100
+Connection ~ 10250 5100
+Wire Wire Line
+	10250 5100 10250 5250
 Wire Bus Line
 	9300 2600 9300 2900
 Wire Bus Line
-	3350 2800 3350 5000
+	3200 2800 3200 5000
 Wire Bus Line
 	10600 3700 10600 4200
@@
 Wire Bus Line
 	5100 1300 5100 2450
+Text Label 5350 800  2    50   ~ 0
+nQ
+Text Label 4000 800  2    50   ~ 0
+nE
+Text Label 2450 4600 2    50   ~ 0
+nQ
+Text Label 2450 2600 2    50   ~ 0
+nQ
+Text Label 2450 4400 2    50   ~ 0
+nE
+Text Label 2450 2400 2    50   ~ 0
+nE
 $EndSCHEMATC
