File: Schematics/74HC/RevC3/CPU2908Executer.sch (KiCad schematic (older format))
At the start: 175 parts, among them U100 TC74VHCT541, U101 74HC153, U102 74HC153, U103 74HC153, U104 74HC153, U105 74HC153, U106 TC74VHCT541, U107 74HC153, U108 TC74VHCT541, U109 74HC153, U110 74HC153, U111 74HC157, U112 74HC157, U113 TC74HC4078, U114 74HC153, U115 74HC139, U116 TC74VHCT541, U120 TC74VHCT04AFT, U123 TC74VHCT04AFT, U26 TC74VHCT04AFT, U27 TC74VHCT04AFT, U30 CD74HC253, U38 CD74HC253, U40 CD74HC253, U44 TC74HC238D, U45 TC74VHC574F, U46 TC74VHC574F, U47 TC74VHC574F, U48 TC74VHC574F, U49 74HC139, U5 CD74HC253, U50 TC74VHC574F, U51 TC74VHC574F, U52 TC74VHC574F, U53 TC74VHC574F, U54 TC74VHC574F, U55 TC74VHC574F, U56 TC74VHCT541, U57 TC74VHCT541, U58 TC74VHC574F, U59 TC74VHC574F, U60 74HC153, U61 74HC153, U62 74HC153, U63 74HC153, U64 TC74VHCT541, U65 TC74VHCT541, U68 74HC153, U69 74HC153, U70 74HC153, U71 74HC153, U72 TC74VHCT541, U75 74HC32, U76 74HC157, U77 74HC157, U78 74HC08D, U79 74HC08D, U80 74HC153, U81 74HC377, U82 74HC377, U83 CD74HC283, U84 CD74HC283, U85 74HC08D, U86 CD74HC283, U87 74HC157, U88 74HC157, U89 74HC08D, U90 SN74AHC86, U91 74HC153, U92 74HC153, U93 CD74HC283, U94 CD74HC283, U95 74HC08D, U96 CD74HC283, U97 74HC153, U98 74HC377, U99 74HC153

Commit message: revA3
Parts:
- removed C104, C60: 0.1uF, Capacitors_SMD:C_0402, symbol Device:C_Small
- removed U123: TC74VHCT04AFT, Housings_SSOP:TSSOP-14_4.4x5mm_Pitch0.65mm, symbol CPU2908CLocal:74HC04
- removed unit 4 of U27
- removed U49: 74HC139, Footprints:MC74HC139ADR2G, symbol CPU2908CLocal:74HC139
- removed U72: TC74VHCT541, digikey-footprints:TSSOP-20_W4.4mm, symbol CPU2908CLocal:74HC541
- added U12: TC74VHCT04AFT, Housings_SSOP:TSSOP-14_4.4x5mm_Pitch0.65mm, symbol CPU2908CLocal:74HC04
- added U49, U66: NC7SZ57, TO_SOT_Packages_SMD:SOT-363_SC-70-6_Handsoldering, symbol CPU2908CLocal:NC7SZ57
- added U67: 74AHC1G04, TO_SOT_Packages_SMD:SOT-23-5, symbol 74xGxx:74AHC1G04
- U81: フィールド4 (none) -> ALU-A
- U82: フィールド4 (none) -> ALU-B
Connections:
- net RO0 is gone; now on net IDB0: U5.7 (1Y)
- net RO1 is gone; now on net IDB1: U5.9 (2Y)
- net RO2 is gone; now on net IDB2: U30.7 (1Y)
- net RO3 is gone; now on net IDB3: U30.9 (2Y)
- net RO4 is gone; now on net IDB4: U38.7 (1Y)
- net RO5 is gone; now on net IDB5: U38.9 (2Y)
- net RO6 is gone; now on net IDB6: U40.7 (1Y)
- net RO7 is gone; now on net IDB7: U40.9 (2Y)
- net +5V: now also U49.5 (VCC), U66.5 (VCC)
- net ALU7: now also U90.2; no longer U90.5
- net ALU_B7: now also U90.5; no longer U90.2
- net BR_SEL2: now also U30.1 (~1OE), U30.15 (~2OE), U38.1 (~1OE), U38.15 (~2OE), U40.1 (~1OE), U40.15 (~2OE), U5.1 (~1OE), U5.15 (~2OE), U67.2
- net BuffSel0: now also U49.1 (I1), U66.6 (I2)
- net BuffSel1: now also U49.6 (I2), U66.1 (I1)
- net GND: now also U12.5, U12.7 (GND), U49.2 (GND), U49.3 (I0), U66.2 (GND), U66.3 (I0), U67.3 (GND); no longer U27.3, U30.1 (~1OE), U30.15 (~2OE), U38.1 (~1OE), U38.15 (~2OE), U40.1 (~1OE), U40.15 (~2OE), U5.1 (~1OE), U5.15 (~2OE)
- net VCC: now also U12.14 (VCC), U67.5 (VCC)
- net at U75.13, U75.9: now also U27.4
- net nBR_SEL2: now reaches U115.15 (~E)
- net nBR_SEL2: now also U67.4
- net at U79.6: now also U27.3
- net at U79.10: now also U90.3; no longer U90.6
- net at U90.10: now also U90.6; no longer U90.3
- net ~B-Active: now reaches U81.1 (~E)
- net ~B-Active: now also U49.4 (Y)
- net ~A-Active: now reaches U82.1 (~E)
- net ~A-Active: now also U66.4 (Y)
- net clk: no longer names the net of U90.11
- no-connect marks 23 -> 18
Other:
- moved on the sheet: U115B, U27B, U90A, U90B
