File: Schematics/74HC/RevC3/CPU2908Sequencer.sch (KiCad schematic (older format))
At the start: 105 parts, among them U10 MC74HC74A, U11 74HC86, U118 MC74ACT125, U12 TC74VHCT04AFT, U122 74HC08D, U123 TC74VHCT04AFT, U13 74HC08D, U14 74HC21, U15 74HC32, U16 74HC153, U17 MC74HC74A, U18 74HC157, U19 TC74VHCT04AFT, U20 SN74HC11D, U21 74HC08D, U22 74HC157, U23 74HC157, U24 74HC32, U25 74HC74, U26 TC74VHCT04AFT, U28 TC74VHCT541, U29 SN74HCT574, U3 TC74VHCT04AFT, U31 NC7SZ58, U32 74HCT273D, U33 74HCT273D, U34 74HCT273D, U35 74HCT273D

Commit message: revA3
Parts:
- removed U122: 74HC08D, digikey-footprints:SOIC-14_W3.9mm, symbol CPU2908CLocal:74HC08
- removed U123, U3: TC74VHCT04AFT, Housings_SSOP:TSSOP-14_4.4x5mm_Pitch0.65mm, symbol CPU2908CLocal:74HC04
- removed unit 5 of U19
- removed unit 4 of U19
- removed unit 2 of U21
- removed unit 3 of U21
- added unit 5 of U12
- added unit 1 of U13
- added U41, U42: 74AHC1G04, TO_SOT_Packages_SMD:SOT-23-5, symbol 74xGxx:74AHC1G04
- added U43: 74AHC1G32, Housings_SSOP:TSOP-5_1.65x3.05mm_Pitch0.95mm, symbol CPU2908C-rescue:74AHC1G32-74xGxx
Connections:
- net OPReg0 is gone; now on net DataIn0: U19.1, U20.5
- net OPReg1 is gone; now on net DataIn1: U16.14 (S0), U26.5
- net OPReg2 is gone; now on net DataIn2: U16.2 (S1), U26.13
- net OPReg3 is gone; now on net DataIn3: U19.3, U20.13
- net OPReg4 is gone; now on net DataIn4: U19.5
- net OPReg5 is gone; now on net DataIn5: U14.10
- net OPReg6 is gone; now on net DataIn6: U14.12
- net OPReg7 is gone; now on net DataIn7: U14.13
- net BusLED0: now also R24.2; no longer D24.2 (A)
- net BusLED1: now also R25.2; no longer D25.2 (A)
- net BusLED2: now also R26.2; no longer D26.2 (A)
- net BusLED3: now also R27.2; no longer D27.2 (A)
- net D23B: now also U29.1 (~OE)
- net DO_JUMP: now also U15.8; no longer U24.6
- net DataIn0: now also U42.2
- net GND: now also U15.12, U15.13, U12.11, U12.7 (GND), U13.7 (GND), U41.3 (GND), U42.3 (GND), U43.3 (GND)
- net GNDD: now also D1.1 (K), D10.1 (K), D11.1 (K), D12.1 (K), D13.1 (K), D14.1 (K), D15.1 (K), D16.1 (K), D17.1 (K), D18.1 (K), D19.1 (K), D2.1 (K), D20.1 (K), D21.1 (K), D22.1 (K), D23.1 (K), D24.1 (K), D25.1 (K), D26.1 (K), D27.1 (K), D3.1 (K), D4.1 (K), D5.1 (K), D6.1 (K), D7.1 (K), D8.1 (K), D9.1 (K); no longer R1.1, R10.1, R11.1, R12.1, R13.1, R14.1, R15.1, R16.1, R17.1, R18.1, R19.1, R2.1, R20.1, R21.1, R22.1, R23.1, R24.1, R25.1, R26.1, R27.1, R3.1, R4.1, R5.1, R6.1, R7.1, R8.1, R9.1
- net JG: now also U41.4
- net RegLED0: now also R1.2; no longer D1.2 (A)
- net RegLED1: now also R2.2; no longer D2.2 (A)
- net RegLED10: now also R11.2; no longer D11.2 (A)
- net RegLED11: now also R12.2; no longer D12.2 (A)
- net RegLED12: now also R13.2; no longer D13.2 (A)
- net RegLED13: now also R14.2; no longer D14.2 (A)
- net RegLED14: now also R15.2; no longer D15.2 (A)
- net RegLED15: now also R16.2; no longer D16.2 (A)
- net RegLED16: now also R17.2; no longer D17.2 (A)
- net RegLED17: now also R18.2; no longer D18.2 (A)
- net RegLED18: now also R19.2; no longer D19.2 (A)
- net RegLED19: now also R20.2; no longer D20.2 (A)
- net RegLED2: now also R3.2; no longer D3.2 (A)
- net RegLED20: now also R21.2; no longer D21.2 (A)
- net RegLED21: now also R22.2; no longer D22.2 (A)
- net RegLED22: now also R23.2; no longer D23.2 (A)
- net RegLED3: now also R4.2; no longer D4.2 (A)
- net RegLED4: now also R5.2; no longer D5.2 (A)
- net RegLED5: now also R6.2; no longer D6.2 (A)
- net RegLED6: now also R7.2; no longer D7.2 (A)
- net RegLED7: now also R8.2; no longer D8.2 (A)
- net RegLED8: now also R9.2; no longer D9.2 (A)
- net RegLED9: now also R10.2; no longer D10.2 (A)
- net S0: now also U13.1
- net VCC: now also U12.14 (VCC), U13.14 (VCC), U41.5 (VCC), U42.5 (VCC), U43.6 (VCC)
- net at U13.12: now also U43.4; no longer U15.11
- net at U22.1 (S), U23.1 (S): now also U24.6; no longer U15.8
- net at U13.10, U19.4: now also U43.2; no longer U15.13
- net at U13.8: now also U15.9; no longer U24.4
- net at U15.3: now also U41.2
- net at U20.12, U20.3, U20.9: now also U43.1; no longer U15.12
- net at U24.1: now also U13.3; no longer U20.6
- net at U24.2: now also U12.3, U14.6; no longer U20.8
- net at U24.3: now also U17.2 (D); no longer U24.5
- net at U11.5, U19.2: no longer U20.11
- net at U15.4: now also U20.6
- net at U15.6: now also U15.10; no longer U17.2 (D)
- net at U13.4, U17.8 (~Q): now also U24.5; no longer U15.10
- net at U17.6 (~Q): now also U24.4, U13.2; no longer U15.9
- new net: U20.11, U42.4
- new net: D1.2 (A), R1.1
- new net: D2.2 (A), R2.1
- new net: D3.2 (A), R3.1
- new net: D4.2 (A), R4.1
- new net: D5.2 (A), R5.1
- new net: D6.2 (A), R6.1
- new net: D7.2 (A), R7.1
- new net: D8.2 (A), R8.1
- new net: D9.2 (A), R9.1
- new net: D10.2 (A), R10.1
- new net: D11.2 (A), R11.1
- new net: D12.2 (A), R12.1
- new net: D13.2 (A), R13.1
- new net: D14.2 (A), R14.1
- new net: D15.2 (A), R15.1
- new net: D16.2 (A), R16.1
- new net: D17.2 (A), R17.1
- new net: D18.2 (A), R18.1
- new net: D19.2 (A), R19.1
- new net: D20.2 (A), R20.1
- new net: D21.2 (A), R21.1
- new net: D22.2 (A), R22.1
- new net: D23.2 (A), R23.1
- new net: D24.2 (A), R24.1
- new net: D25.2 (A), R25.1
- new net: D26.2 (A), R26.1
- new net: D27.2 (A), R27.1
- new net: U15.5, U20.8
- no-connect marks 21 -> 22
Other:
- moved on the sheet: D1, R1, R10, R11, R12, R13, R14, R15, R16, R17, R18, R19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
