File: Schematics/74HC/RevCP4/CPU2908Executer.sch (KiCad schematic (older format))
At the start: 174 parts, among them U100 TC74VHCT541, U101 74HC153, U102 74HC153, U103 74HC153, U104 74HC153, U105 74HC153, U106 TC74VHCT541, U107 74HC153, U108 TC74VHCT541, U109 74HC153, U110 74HC153, U111 74HC157, U112 74HC157, U113 TC74HC4078, U114 74HC153, U115 74HC139, U116 TC74VHCT541, U12 TC74VHCT04AFT, U120 TC74VHCT04AFT, U27 TC74VHCT04AFT, U30 CD74HC253, U38 CD74HC253, U40 CD74HC253, U44 TC74HC238D, U45 TC74VHC574F, U46 TC74VHC574F, U47 TC74VHC574F, U48 TC74VHC574F, U49 NC7SZ57, U5 CD74HC253, U50 TC74VHC574F, U51 TC74VHC574F, U52 TC74VHC574F, U53 TC74VHC574F, U54 TC74VHC574F, U55 TC74VHC574F, U56 TC74VHCT541, U57 TC74VHCT541, U58 TC74VHC574F, U59 TC74VHC574F, U60 74HC153, U61 74HC153, U62 74HC153, U63 74HC153, U64 TC74VHCT541, U65 TC74VHCT541, U66 NC7SZ57, U67 74AHC1G04, U68 74HC153, U69 74HC153, U70 74HC153, U71 74HC153, U72 74HC139, U75 74HC32, U76 74HC157, U77 74HC157, U78 74HC08D, U79 74HC08D, U80 74HC153, U81 74HC377, U82 74HC377, U83 CD74HC283, U84 CD74HC283, U85 74HC08D, U86 CD74HC283, U87 74HC157, U88 74HC157, U89 74HC08D, U90 SN74AHC86, U91 74HC153, U92 74HC153, U93 CD74HC283, U94 CD74HC283, U95 74HC08D, U96 CD74HC283, U97 74HC153, U98 74HC377, U99 74HC153

Commit message: インストラクション変更
Changed lines of the file:
@@
 U 1 1 782541A6
 P 13350 9400
-F 0 "U90" H 13350 9725 50  0000 C CNN
-F 1 "SN74AHC86" H 13350 9634 50  0000 C CNN
+F 0 "U90" H 13550 9700 50  0000 C CNN
+F 1 "SN74AHC86" H 13300 10000 50  0000 C CNN
 F 2 "Footprints:SN74AHC86D" H 13350 9400 50  0001 C CNN
 F 3 "" H 13350 9400 50  0000 C CNN
@@
 U 2 1 785E8395
 P 13350 9000
-F 0 "U90" H 13350 8777 50  0000 C CNN
-F 1 "SN74AHC86" H 13350 8686 50  0000 C CNN
+F 0 "U90" H 13350 8400 50  0000 C CNN
+F 1 "SN74AHC86" H 13350 8300 50  0000 C CNN
 F 2 "Footprints:SN74AHC86D" H 13350 9000 50  0001 C CNN
 F 3 "" H 13350 9000 50  0000 C CNN
