File: Schematics/MachXO2/FT2232D.sch (KiCad schematic (older format))
At the start: 39 parts, among them J3 USB_B_Micro, U2 FT2232D, U4 93C56, X2 6.00MHz

Commit message: Update Schematic
Parts:
- U4: footprint Housings_SOIC:SO-8_5.3x6.2mm_Pitch1.27mm -> Housings_SOIC:SOIC-8_3.9x4.9mm_Pitch1.27mm
Changed lines of the file:
@@
 F 0 "U4" H 3950 5431 50  0000 C CNN
 F 1 "93C56" H 3700 4650 50  0000 C CNN
-F 2 "Housings_SOIC:SO-8_5.3x6.2mm_Pitch1.27mm" H 3950 4950 50  0001 C CNN
+F 2 "Housings_SOIC:SOIC-8_3.9x4.9mm_Pitch1.27mm" H 3950 4950 50  0001 C CNN
 F 3 "http://ww1.microchip.com/downloads/en/DeviceDoc/20001749K.pdf" H 3950 4950 50  0001 C CNN
 	1    3950 4950

Commit message: Add schematic Rev C3.
Parts:
- FB1: footprint Capacitors_SMD:C_0603 -> Capacitors_SMD:C_0805; symbol Device:Ferrite_Bead -> o2_breakout-rescue:Ferrite_Bead-Device
- J3: symbol Connector:USB_B_Micro -> o2_breakout-rescue:USB_B_Micro-Connector
- R4, R5, R6: footprint Capacitors_SMD:C_0805 -> Capacitors_SMD:C_0603
- X2: symbol Oscillator:SG-8002CA -> o2_breakout-rescue:SG-8002CA-Oscillator
Changed lines of the file:
@@
 $EndComp
 $Comp
-L Connector:USB_B_Micro J3
+L o2_breakout-rescue:USB_B_Micro-Connector J3
 U 1 1 5E6AAFE7
 P 3450 1700
+AR Path="/5E6AAFE7" Ref="J3"  Part="1"
+AR Path="/5E6A6650/5E6AAFE7" Ref="J3"  Part="1"
 F 0 "J3" H 3507 2167 50  0000 C CNN
 F 1 "USB_B_Micro" H 3507 2076 50  0000 C CNN
@@
 Connection ~ 4450 5050
 $Comp
-L Oscillator:SG-8002CA X?
+L o2_breakout-rescue:SG-8002CA-Oscillator X?
 U 1 1 5DC12BA3
 P 3550 3850
@@
 F 0 "R6" V 4400 3500 50  0000 C CNN
 F 1 "1.5K" V 4350 3350 50  0000 C CNN
-F 2 "Capacitors_SMD:C_0805" V 4380 3350 50  0001 C CNN
+F 2 "Capacitors_SMD:C_0603" V 4380 3350 50  0001 C CNN
 F 3 "~" H 4450 3350 50  0001 C CNN
 	1    4450 3350
@@
 F 0 "R4" V 4093 2950 50  0000 C CNN
 F 1 "27" V 4184 2950 50  0000 C CNN
-F 2 "Capacitors_SMD:C_0805" V 4230 2950 50  0001 C CNN
+F 2 "Capacitors_SMD:C_0603" V 4230 2950 50  0001 C CNN
 F 3 "~" H 4300 2950 50  0001 C CNN
 	1    4300 2950
@@
 F 0 "R5" V 4250 3000 50  0000 C CNN
 F 1 "27" V 4200 3150 50  0000 C CNN
-F 2 "Capacitors_SMD:C_0805" V 4230 3150 50  0001 C CNN
+F 2 "Capacitors_SMD:C_0603" V 4230 3150 50  0001 C CNN
 F 3 "~" H 4300 3150 50  0001 C CNN
 	1    4300 3150
@@
 $EndComp
 $Comp
-L Device:Ferrite_Bead FB1
+L o2_breakout-rescue:Ferrite_Bead-Device FB1
 U 1 1 5DC565F5
 P 4650 1500
 F 0 "FB1" V 4376 1500 50  0000 C CNN
 F 1 "Ferrite_Bead" V 4467 1500 50  0000 C CNN
-F 2 "Capacitors_SMD:C_0603" V 4580 1500 50  0001 C CNN
+F 2 "Capacitors_SMD:C_0805" V 4580 1500 50  0001 C CNN
 F 3 "~" H 4650 1500 50  0001 C CNN
 	1    4650 1500

Commit message: Update Schematics
Parts:
- added D7, D8: LED, Capacitors_SMD:C_0402, symbol CPU2908CLocal:LED
- added R27, R28: 22K, Capacitors_SMD:C_0402, symbol CPU2908CLocal:R
Connections:
- net +3V3: now also R27.1, R28.1
- net ~TxLED: now reaches U2.27 (BCBUS3)
- net ~TxLED: now also D8.1 (K)
- net ~RxLED: now reaches U2.28 (BCBUS2)
- net ~RxLED: now also D7.1 (K)
- new net: D8.2 (A), R28.2
- new net: D7.2 (A), R27.2
- no-connect marks 21 -> 19
Changed lines of the file:
@@
 $EndComp
 Wire Wire Line
-	6700 3850 7100 3850
-Wire Wire Line
-	6700 3950 7100 3950
-Wire Wire Line
-	6700 4050 7100 4050
-Wire Wire Line
-	6700 4150 7100 4150
-Text HLabel 7100 3850 2    50   Output ~ 0
+	6700 3850 6850 3850
+Wire Wire Line
+	6700 3950 6850 3950
+Wire Wire Line
+	6700 4050 6850 4050
+Wire Wire Line
+	6700 4150 6850 4150
+Text HLabel 6850 3850 2    50   Output ~ 0
 TxD_FT
-Text HLabel 7100 3950 2    50   Input ~ 0
+Text HLabel 6850 3950 2    50   Input ~ 0
 RxD_FT
-Text HLabel 7100 4050 2    50   Output ~ 0
+Text HLabel 6850 4050 2    50   Output ~ 0
 ~RTS_FT
-Text HLabel 7100 4150 2    50   Input ~ 0
+Text HLabel 6850 4150 2    50   Input ~ 0
 ~CTS_FT
 Text HLabel 7300 2350 2    50   Output ~ 0
@@
 NoConn ~ 6700 4750
 NoConn ~ 6700 4850
-NoConn ~ 6700 4950
-NoConn ~ 6700 5050
 NoConn ~ 6700 5150
 Wire Wire Line
@@
 	1    0    0    -1
 $EndComp
+$Comp
+L CPU2908CLocal:LED D8
+U 1 1 5E4339D9
+P 7700 4700
+F 0 "D8" V 7739 4583 50  0000 R CNN
+F 1 "LED" V 7648 4583 50  0000 R CNN
+F 2 "Capacitors_SMD:C_0402" H 7700 4700 50  0001 C CNN
+F 3 "~" H 7700 4700 50  0001 C CNN
+	1    7700 4700
+	0    -1   -1   0
+$EndComp
+$Comp
+L CPU2908CLocal:LED D7
+U 1 1 5E4350D2
+P 7450 4700
+F 0 "D7" V 7489 4583 50  0000 R CNN
+F 1 "LED" V 7398 4583 50  0000 R CNN
+F 2 "Capacitors_SMD:C_0402" H 7450 4700 50  0001 C CNN
+F 3 "~" H 7450 4700 50  0001 C CNN
+	1    7450 4700
+	0    -1   -1   0
+$EndComp
+$Comp
+L power:+3V3 #PWR024
+U 1 1 5E4533E1
+P 7700 4050
+F 0 "#PWR024" H 7700 3900 50  0001 C CNN
+F 1 "+3V3" H 7715 4223 50  0000 C CNN
+F 2 "" H 7700 4050 50  0001 C CNN
+F 3 "" H 7700 4050 50  0001 C CNN
+	1    7700 4050
+	1    0    0    -1
+$EndComp
+$Comp
+L CPU2908CLocal:R R28
+U 1 1 5E4533E7
+P 7700 4350
+F 0 "R28" H 7770 4396 50  0000 L CNN
+F 1 "22K" H 7770 4305 50  0000 L CNN
+F 2 "Capacitors_SMD:C_0402" V 7630 4350 50  0001 C CNN
+F 3 "~" H 7700 4350 50  0001 C CNN
+	1    7700 4350
+	1    0    0    -1
+$EndComp
+$Comp
+L CPU2908CLocal:R R27
+U 1 1 5E4533ED
+P 7450 4350
+F 0 "R27" H 7520 4396 50  0000 L CNN
+F 1 "22K" H 7520 4305 50  0000 L CNN
+F 2 "Capacitors_SMD:C_0402" V 7380 4350 50  0001 C CNN
+F 3 "~" H 7450 4350 50  0001 C CNN
+	1    7450 4350
+	1    0    0    -1
+$EndComp
+Wire Wire Line
+	7700 4200 7700 4100
+Wire Wire Line
+	7450 4200 7450 4100
+Wire Wire Line
+	7450 4500 7450 4550
+Wire Wire Line
+	7450 4100 7700 4100
+Connection ~ 7700 4100
+Wire Wire Line
+	7700 4100 7700 4050
+Wire Wire Line
+	7700 4500 7700 4550
+Wire Wire Line
+	6700 4950 7450 4950
+Wire Wire Line
+	7450 4950 7450 4850
+Wire Wire Line
+	6700 5050 7700 5050
+Wire Wire Line
+	7700 5050 7700 4850
+Text Label 6850 4950 0    50   ~ 0
+~RxLED
+Text Label 6850 5050 0    50   ~ 0
+~TxLED
 $EndSCHEMATC

Commit message: BUG Fix.
Other:
- moved on the sheet: D7, D8, R27, R28
Changed lines of the file:
@@
 $EndComp
 Wire Wire Line
-	6700 3850 6850 3850
-Wire Wire Line
-	6700 3950 6850 3950
-Wire Wire Line
-	6700 4050 6850 4050
-Wire Wire Line
-	6700 4150 6850 4150
-Text HLabel 6850 3850 2    50   Output ~ 0
+	6700 3850 7550 3850
+Wire Wire Line
+	6700 3950 7550 3950
+Wire Wire Line
+	6700 4050 7550 4050
+Wire Wire Line
+	6700 4150 7550 4150
+Text HLabel 7550 3850 2    50   Output ~ 0
 TxD_FT
-Text HLabel 6850 3950 2    50   Input ~ 0
+Text HLabel 7550 3950 2    50   Input ~ 0
 RxD_FT
-Text HLabel 6850 4050 2    50   Output ~ 0
+Text HLabel 7550 4050 2    50   Output ~ 0
 ~RTS_FT
-Text HLabel 6850 4150 2    50   Input ~ 0
+Text HLabel 7550 4150 2    50   Input ~ 0
 ~CTS_FT
 Text HLabel 7300 2350 2    50   Output ~ 0
@@
 L CPU2908CLocal:LED D8
 U 1 1 5E4339D9
-P 7700 4700
-F 0 "D8" V 7739 4583 50  0000 R CNN
-F 1 "LED" V 7648 4583 50  0000 R CNN
-F 2 "Capacitors_SMD:C_0402" H 7700 4700 50  0001 C CNN
-F 3 "~" H 7700 4700 50  0001 C CNN
-	1    7700 4700
+P 8600 4700
+F 0 "D8" V 8639 4583 50  0000 R CNN
+F 1 "LED" V 8548 4583 50  0000 R CNN
+F 2 "Capacitors_SMD:C_0402" H 8600 4700 50  0001 C CNN
+F 3 "~" H 8600 4700 50  0001 C CNN
+	1    8600 4700
 	0    -1   -1   0
 $EndComp
@@
 L CPU2908CLocal:LED D7
 U 1 1 5E4350D2
-P 7450 4700
-F 0 "D7" V 7489 4583 50  0000 R CNN
-F 1 "LED" V 7398 4583 50  0000 R CNN
-F 2 "Capacitors_SMD:C_0402" H 7450 4700 50  0001 C CNN
-F 3 "~" H 7450 4700 50  0001 C CNN
-	1    7450 4700
+P 8350 4700
+F 0 "D7" V 8389 4583 50  0000 R CNN
+F 1 "LED" V 8298 4583 50  0000 R CNN
+F 2 "Capacitors_SMD:C_0402" H 8350 4700 50  0001 C CNN
+F 3 "~" H 8350 4700 50  0001 C CNN
+	1    8350 4700
 	0    -1   -1   0
 $EndComp
@@
 L power:+3V3 #PWR024
 U 1 1 5E4533E1
-P 7700 4050
-F 0 "#PWR024" H 7700 3900 50  0001 C CNN
-F 1 "+3V3" H 7715 4223 50  0000 C CNN
-F 2 "" H 7700 4050 50  0001 C CNN
-F 3 "" H 7700 4050 50  0001 C CNN
-	1    7700 4050
+P 8600 4050
+F 0 "#PWR024" H 8600 3900 50  0001 C CNN
+F 1 "+3V3" H 8615 4223 50  0000 C CNN
+F 2 "" H 8600 4050 50  0001 C CNN
+F 3 "" H 8600 4050 50  0001 C CNN
+	1    8600 4050
 	1    0    0    -1
 $EndComp
@@
 L CPU2908CLocal:R R28
 U 1 1 5E4533E7
-P 7700 4350
-F 0 "R28" H 7770 4396 50  0000 L CNN
-F 1 "22K" H 7770 4305 50  0000 L CNN
-F 2 "Capacitors_SMD:C_0402" V 7630 4350 50  0001 C CNN
-F 3 "~" H 7700 4350 50  0001 C CNN
-	1    7700 4350
+P 8600 4350
+F 0 "R28" H 8670 4396 50  0000 L CNN
+F 1 "22K" H 8670 4305 50  0000 L CNN
+F 2 "Capacitors_SMD:C_0402" V 8530 4350 50  0001 C CNN
+F 3 "~" H 8600 4350 50  0001 C CNN
+	1    8600 4350
 	1    0    0    -1
 $EndComp
@@
 L CPU2908CLocal:R R27
 U 1 1 5E4533ED
-P 7450 4350
-F 0 "R27" H 7520 4396 50  0000 L CNN
-F 1 "22K" H 7520 4305 50  0000 L CNN
-F 2 "Capacitors_SMD:C_0402" V 7380 4350 50  0001 C CNN
-F 3 "~" H 7450 4350 50  0001 C CNN
-	1    7450 4350
-	1    0    0    -1
-$EndComp
-Wire Wire Line
-	7700 4200 7700 4100
-Wire Wire Line
-	7450 4200 7450 4100
-Wire Wire Line
-	7450 4500 7450 4550
-Wire Wire Line
-	7450 4100 7700 4100
-Connection ~ 7700 4100
-Wire Wire Line
-	7700 4100 7700 4050
-Wire Wire Line
-	7700 4500 7700 4550
-Wire Wire Line
-	6700 4950 7450 4950
-Wire Wire Line
-	7450 4950 7450 4850
-Wire Wire Line
-	6700 5050 7700 5050
-Wire Wire Line
-	7700 5050 7700 4850
+P 8350 4350
+F 0 "R27" H 8420 4396 50  0000 L CNN
+F 1 "22K" H 8420 4305 50  0000 L CNN
+F 2 "Capacitors_SMD:C_0402" V 8280 4350 50  0001 C CNN
+F 3 "~" H 8350 4350 50  0001 C CNN
+	1    8350 4350
+	1    0    0    -1
+$EndComp
+Wire Wire Line
+	8600 4200 8600 4100
+Wire Wire Line
+	8350 4200 8350 4100
+Wire Wire Line
+	8350 4500 8350 4550
+Wire Wire Line
+	8350 4100 8600 4100
+Connection ~ 8600 4100
+Wire Wire Line
+	8600 4100 8600 4050
+Wire Wire Line
+	8600 4500 8600 4550
+Wire Wire Line
+	6700 4950 8350 4950
+Wire Wire Line
+	8350 4950 8350 4850
+Wire Wire Line
+	6700 5050 8600 5050
+Wire Wire Line
+	8600 5050 8600 4850
 Text Label 6850 4950 0    50   ~ 0
 ~RxLED
