File: Schematics/MachXO2/SDCARD.sch (KiCad schematic (older format))
At the start: 21 parts, among them J4 DM3AT-SF-PEJM5, U7 PCF2129AT, U9 AT25xxx

Commit message: Update Schematic
Parts:
- U9: footprint Package_SO:SOIC-8_5.23x5.23mm_P1.27mm -> Housings_SOIC:SOIC-8_3.9x4.9mm_Pitch1.27mm
Changed lines of the file:
@@
 F 0 "U9" H 4250 5350 50  0000 C CNN
 F 1 "AT25xxx" H 4700 4850 50  0000 C CNN
-F 2 "Package_SO:SOIC-8_5.23x5.23mm_P1.27mm" H 4500 5100 50  0001 C CNN
+F 2 "Housings_SOIC:SOIC-8_3.9x4.9mm_Pitch1.27mm" H 4500 5100 50  0001 C CNN
 F 3 "http://ww1.microchip.com/downloads/en/DeviceDoc/Atmel-8707-SEEPROM-AT25010B-020B-040B-Datasheet.pdf" H 4500 5100 50  0001 C CNN
 	1    4500 5100

Commit message: Add schematic Rev C3.
Parts:
- U7: symbol Timer_RTC:PCF2129AT -> o2_breakout-rescue:PCF2129AT-Timer_RTC
Changed lines of the file:
@@
 SD_CLK
 $Comp
-L Timer_RTC:PCF2129AT U7
+L o2_breakout-rescue:PCF2129AT-Timer_RTC U7
 U 1 1 5DF2754E
 P 6200 3900
+AR Path="/5DF2754E" Ref="U7"  Part="1"
+AR Path="/5DD58257/5DF2754E" Ref="U7"  Part="1"
 F 0 "U7" H 5950 4450 50  0000 L CNN
 F 1 "PCF2129AT" H 6000 3250 50  0000 L CNN

Commit message: Update BreakOut Schematic.
Parts:
- R8: value 2.2K -> 10K; footprint Capacitors_SMD:C_0603 -> Capacitors_SMD:C_0402
Connections:
- no-connect marks 5 -> 4
Changed lines of the file:
@@
 P 5550 1650
 F 0 "R8" H 5620 1696 50  0000 L CNN
-F 1 "2.2K" H 5620 1605 50  0000 L CNN
-F 2 "Capacitors_SMD:C_0603" V 5480 1650 50  0001 C CNN
+F 1 "10K" H 5620 1605 50  0000 L CNN
+F 2 "Capacitors_SMD:C_0402" V 5480 1650 50  0001 C CNN
 F 3 "~" H 5550 1650 50  0001 C CNN
 	1    5550 1650
@@
 U 1 1 5E9F8758
 P 7100 4450
-F 0 "C30" V 7396 4322 50  0000 R CNN
-F 1 "DCK-3R3E224-E" V 7400 4100 50  0000 R CNN
+F 0 "C30" V 7450 4400 50  0000 R CNN
+F 1 "DCK-3R3E224-E" V 7250 4700 50  0000 R CNN
 F 2 "digikey-footprints:DCK-3R3E224-E" H 7450 4500 50  0001 L CNN
 F 3 "http://www.21datasheet.com/index/download_pdf/id/Pn5roYB58yeq" H 7450 4400 50  0001 L CNN
@@
 Text HLabel 4800 4100 0    50   Output ~ 0
 RTC_CLK
-NoConn ~ 6650 3700
 NoConn ~ 5750 4000
 Wire Wire Line
@@
 U 1 1 5E3C94A0
 P 6900 4150
-F 0 "C24" H 6950 4350 50  0000 L CNN
-F 1 "0.1uF" H 6950 4300 50  0000 L CNN
+F 0 "C24" H 6750 4350 50  0000 L CNN
+F 1 "0.1uF" H 6750 4250 50  0000 L CNN
 F 2 "Capacitors_SMD:C_0402" H 6938 4000 50  0001 C CNN
 F 3 "~" H 6900 4150 50  0001 C CNN

Commit message: Update schematics
Parts:
- added R29: 10K, Capacitors_SMD:C_0402, symbol CPU2908CLocal:R
Connections:
- net +3V3: now also R29.1
- net ~SD_CS: now also R29.2
- net DAT2_NC: now reaches J4.1 (DAT2)
- net DAT1_NC: now reaches J4.8 (DAT1)
- no-connect marks 4 -> 2
Changed lines of the file:
@@
 Connection ~ 5550 1950
 Wire Wire Line
-	5550 1950 5400 1950
-NoConn ~ 5700 2150
-NoConn ~ 5700 2050
+	5550 1950 5300 1950
 $Comp
 L Device:C C23
@@
 $EndComp
 Wire Wire Line
-	4200 2250 5700 2250
+	4200 2250 4700 2250
 Text HLabel 4200 2250 0    50   Input ~ 0
 ~SD_CS
@@
 	4900 2350 5700 2350
 Wire Wire Line
-	5400 1950 5400 2150
-Wire Wire Line
-	5400 2150 5100 2150
+	5300 1950 5300 2150
+Wire Wire Line
+	5300 2150 5100 2150
 Text HLabel 4200 2150 0    50   Input ~ 0
 SD_DO
@@
 Wire Wire Line
 	7200 3500 7850 3500
+Wire Wire Line
+	5450 2050 5700 2050
+Wire Wire Line
+	5450 2150 5700 2150
+Text Label 5450 2050 0    50   ~ 0
+DAT1_NC
+Text Label 5450 2150 0    50   ~ 0
+DAT2_NC
+$Comp
+L CPU2908CLocal:R R29
+U 1 1 5E6CE917
+P 4700 1900
+F 0 "R29" H 4770 1946 50  0000 L CNN
+F 1 "10K" H 4770 1855 50  0000 L CNN
+F 2 "Capacitors_SMD:C_0402" V 4630 1900 50  0001 C CNN
+F 3 "~" H 4700 1900 50  0001 C CNN
+	1    4700 1900
+	1    0    0    -1
+$EndComp
+Wire Wire Line
+	4700 2050 4700 2250
+Connection ~ 4700 2250
+Wire Wire Line
+	4700 2250 5700 2250
+Wire Wire Line
+	4700 1750 4700 1350
+Wire Wire Line
+	4700 1350 4900 1350
 $EndSCHEMATC

Commit message: revA3
Parts:
- removed D1: D, Capacitors_SMD:C_0603_HandSoldering, symbol Device:D
- added D9: LED, Capacitors_SMD:C_0603, symbol CPU2908CLocal:LED
- added R30: 10K, Capacitors_SMD:C_0402, symbol CPU2908CLocal:R
- added R31: 47K, Capacitors_SMD:C_0402, symbol CPU2908CLocal:R
- added U6: MAX40200AUK, TO_SOT_Packages_SMD:SOT-23-5, symbol Analog_Switch:MAX40200AUK
- C23: value 10uF -> 47uF; footprint Capacitors_SMD:C_0805 -> Capacitors_SMD:C_1210
- R15: value 1R0 -> 33
- R7: value 1R0 -> 33; footprint Capacitors_SMD:C_0603 -> Capacitors_SMD:C_0805
Connections:
- net +3V3: now also D9.2 (A), R30.1, U6.1 (VDD), U6.3 (EN)
- net GND: now also U6.2 (GND)
- net VBat: no longer C34.1
- net ~PROM_CS: now also R30.2
- net ~SD_CS: now also R31.2
- net RTCVdd: now reaches C21.1, C25.1, R9.1, U7.20 (Vdd)
- net ~WP: now reaches R14.2, U9.3 (~WP)
- net ~HOLD: now reaches R13.2, U9.7 (~HOLD)
- net at R15.1: now also C34.1, U6.5 (OUT)
- new net: D9.1 (K), R31.1
Other:
- moved on the sheet: R13, R14, R15
