File: Schematics/MachXO2/o2_breakout.sch (KiCad schematic (older format))
At the start: 37 parts, among them J1 Conn_02x20_Odd_Even, J2 Conn_02x20_Odd_Even, SW1 USER, SW2 Reset, U1 LCMXO2-2000HC-4TG100C, U3 TCM809, U5 CY7C1010, U8 74AHC1G08, X1 19.6608MHz

Commit message: revA3
Parts:
- removed D4, D6: LED, Capacitors_SMD:C_0603, symbol CPU2908CLocal:LED
- removed R20: 47K, Capacitors_SMD:C_0402, symbol CPU2908CLocal:R
- added C26: 0.1uF, Capacitors_SMD:C_0402, symbol Device:C
- added D10: LED, Capacitors_SMD:C_0603, symbol CPU2908CLocal:LED
- added R32: 47K, Capacitors_SMD:C_0402, symbol CPU2908CLocal:R
- added SW3: SW_Push, digikey-footprints:SMD-2_3.2x1.5mm, symbol Switch:SW_Push
- R18: value 47K -> 10K
Connections:
- net +3V3: now also R18.1, R32.1
- net GND: now also C26.2, SW3.1; no longer R18.2
- net ~CE: now also D10.1 (K)
- net INT: now reaches U1.21 (PL12B)
- net INT: now also R18.2, C26.1, SW3.2
- new net: D10.2 (A), R32.2
- no-connect marks 13 -> 12
Other:
- moved on the sheet: H1, H2, H3, H4, JP2, R25, X1

Commit message: Update Gerber Data to RevA5
Connections:
- net FT_Reset: no longer names the net of U3.2 (~RESET~), U8.1
Changed lines of the file:
@@
 F0 "FT2232D" 50
 F1 "FT2232D.sch" 50
-F2 "nReset" I R 8850 4850 50
-F3 "TxD_FT" O R 8850 3950 50
-F4 "RxD_FT" I R 8850 4050 50
-F5 "TCK_FT" O R 8850 4350 50
-F6 "TDI_FT" O R 8850 4450 50
-F7 "TDO_FT" I R 8850 4550 50
-F8 "TMS_FT" O R 8850 4650 50
-F9 "~RTS_FT" O R 8850 4150 50
-F10 "~CTS_FT" I R 8850 4250 50
+F2 "TxD_FT" O R 8850 3950 50
+F3 "RxD_FT" I R 8850 4050 50
+F4 "TCK_FT" O R 8850 4350 50
+F5 "TDI_FT" O R 8850 4450 50
+F6 "TDO_FT" I R 8850 4550 50
+F7 "TMS_FT" O R 8850 4650 50
+F8 "~RTS_FT" O R 8850 4150 50
+F9 "~CTS_FT" I R 8850 4250 50
 $EndSheet
 Text Label 10500 1450 2    50   ~ 0
@@
 	10500 5650 11050 5650
 Wire Wire Line
-	9250 1550 9350 1550
-Text Label 9700 1700 2    50   ~ 0
-FT_Reset
-Text Label 9350 4850 2    50   ~ 0
-FT_Reset
-Wire Wire Line
-	8850 4850 9350 4850
-Connection ~ 9350 1550
-Wire Wire Line
-	9350 1550 9600 1550
-Wire Wire Line
-	9350 1550 9350 1700
-Wire Wire Line
-	9350 1700 9700 1700
-Wire Wire Line
 	5100 5300 5600 5300
 Wire Wire Line
@@
 Wire Bus Line
 	6050 1100 6050 3500
+Wire Wire Line
+	9250 1550 9600 1550
 $EndSCHEMATC
